File: pcb/rf.sch (KiCad schematic (older format))
At the start: 32 parts, among them J3 Conn_Coaxial, U3 nRF24L01P, U4 RFX2401C, Y2 16 MHz

Commit message: add more decoupling caps and notes
Parts:
- C17: renamed from C13; value 10 uF -> 4.7 uF
- renumbered C11 to C15, C12 to C16, C14 to C18, C15 to C19, C16 to C20, C17 to C21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
Other:
- moved on the sheet: C15, C16, C20, R7
